File: Black-Smoke-Probe.kicad_sch (KiCad schematic)
At the start: 58 parts, among them J1 Conn_ARM_JTAG_SWD_10, J2 USB_C_Receptacle_USB2.0_14P, J3 MCU_BOOT, J5 MCU_SWD, U1 STM32F103CBUx, U2 74LVC2T45DC, U3 74LVC2T45DC, U4 74LVC2T45DC, U5 USBLC6-2P6, U6 NCP662SQ33, U7 DMG1024UV-7, Y2 8MHz

Commit message: first changes for v1.1
- schematic corrections
- new layout with 4 layer PCB
Parts:
- removed J1: Conn_ARM_JTAG_SWD_10, Connector_PinSocket_1.27mm:PinSocket_2x05_P1.27mm_Vertical_SMD, symbol Connector:Conn_ARM_JTAG_SWD_10
- removed J5: MCU_SWD, Connector_PinHeader_2.54mm:PinHeader_1x05_P2.54mm_Vertical, symbol Connector_Generic:Conn_01x05
- removed U1: STM32F103CBUx, Package_DFN_QFN:QFN-48-1EP_7x7mm_P0.5mm_EP5.6x5.6mm, symbol MCU_ST_STM32F1:STM32F103CBUx
- removed U5: USBLC6-2P6, Package_TO_SOT_SMD:SOT-666, symbol Power_Protection:USBLC6-2P6
- removed U6: NCP662SQ33, Package_TO_SOT_SMD:SC-82AB, symbol Regulator_Linear:NCP662SQ33
- added J3: SWD_TagConnect, Connector:Tag-Connect_TC2030-IDC-NL_2x03_P1.27mm_Vertical, symbol Connector:Conn_ARM_SWD_TagConnect_TC2030-NL
- added J4: Conn_ARM_JTAG_SWD_10, Connector_PinHeader_1.27mm:PinHeader_2x05_P1.27mm_Vertical_SMD, symbol Connector:Conn_ARM_JTAG_SWD_10
- added TP6: TestPoint, TestPoint:TestPoint_Pad_D1.0mm, symbol Connector:TestPoint
- added U1: USBLC6-2SC6, Package_TO_SOT_SMD:SOT-23-6, symbol Power_Protection:USBLC6-2SC6
- added U2: AZ1117-3.3, Package_TO_SOT_SMD:SOT-89-3, symbol Regulator_Linear:AZ1117-3.3
- added U3: STM32F103CBTx, Package_QFP:LQFP-48_7x7mm_P0.5mm, symbol MCU_ST_STM32F1:STM32F103CBTx
- C1: renamed from C7; footprint Capacitor_SMD:C_0603_1608Metric_Pad1.08x0.95mm_HandSolder -> Capacitor_SMD:C_0603_1608Metric
- C10: renamed from C9; footprint Capacitor_SMD:C_0603_1608Metric_Pad1.08x0.95mm_HandSolder -> Capacitor_SMD:C_0603_1608Metric
- C11: renamed from C1; footprint Capacitor_SMD:C_0603_1608Metric_Pad1.08x0.95mm_HandSolder -> Capacitor_SMD:C_0603_1608Metric
- C12: renamed from C3; footprint Capacitor_SMD:C_0603_1608Metric_Pad1.08x0.95mm_HandSolder -> Capacitor_SMD:C_0603_1608Metric
- C13: renamed from C5; footprint Capacitor_SMD:C_0603_1608Metric_Pad1.08x0.95mm_HandSolder -> Capacitor_SMD:C_0603_1608Metric
- C14: renamed from C2; footprint Capacitor_SMD:C_0603_1608Metric_Pad1.08x0.95mm_HandSolder -> Capacitor_SMD:C_0603_1608Metric
- C15: renamed from C4; footprint Capacitor_SMD:C_0603_1608Metric_Pad1.08x0.95mm_HandSolder -> Capacitor_SMD:C_0603_1608Metric
- C16: renamed from C6; footprint Capacitor_SMD:C_0603_1608Metric_Pad1.08x0.95mm_HandSolder -> Capacitor_SMD:C_0603_1608Metric
- C2: renamed from C15; footprint Capacitor_SMD:C_0603_1608Metric_Pad1.08x0.95mm_HandSolder -> Capacitor_SMD:C_0603_1608Metric
- C3: renamed from C16; footprint Capacitor_SMD:C_0603_1608Metric_Pad1.08x0.95mm_HandSolder -> Capacitor_SMD:C_0603_1608Metric
- C4: renamed from C13; value 1uF -> 10uF; footprint Capacitor_SMD:C_0603_1608Metric_Pad1.08x0.95mm_HandSolder -> Capacitor_SMD:C_0603_1608Metric
- C5: renamed from C14; value 1uF -> 22uF; footprint Capacitor_SMD:C_0603_1608Metric_Pad1.08x0.95mm_HandSolder -> Capacitor_SMD:C_0603_1608Metric
- C6: renamed from C12; footprint Capacitor_SMD:C_0603_1608Metric_Pad1.08x0.95mm_HandSolder -> Capacitor_SMD:C_0603_1608Metric
- C7: renamed from C10; footprint Capacitor_SMD:C_0603_1608Metric_Pad1.08x0.95mm_HandSolder -> Capacitor_SMD:C_0603_1608Metric
- C8: renamed from C11; footprint Capacitor_SMD:C_0603_1608Metric_Pad1.08x0.95mm_HandSolder -> Capacitor_SMD:C_0603_1608Metric
- C9: renamed from C8; footprint Capacitor_SMD:C_0603_1608Metric_Pad1.08x0.95mm_HandSolder -> Capacitor_SMD:C_0603_1608Metric
- D1: renamed from D4; footprint LED_SMD:LED_0603_1608Metric_Pad1.05x0.95mm_HandSolder -> LED_SMD:LED_0603_1608Metric
- D2: renamed from D1; footprint LED_SMD:LED_0603_1608Metric_Pad1.05x0.95mm_HandSolder -> LED_SMD:LED_0603_1608Metric
- D3: renamed from D2; footprint LED_SMD:LED_0603_1608Metric_Pad1.05x0.95mm_HandSolder -> LED_SMD:LED_0603_1608Metric
- D4: renamed from D3; footprint LED_SMD:LED_0603_1608Metric_Pad1.05x0.95mm_HandSolder -> LED_SMD:LED_0603_1608Metric
- R1: renamed from R10; footprint Resistor_SMD:R_0603_1608Metric_Pad0.98x0.95mm_HandSolder -> Resistor_SMD:R_0603_1608Metric
- R10: renamed from R9; footprint Resistor_SMD:R_0603_1608Metric_Pad0.98x0.95mm_HandSolder -> Resistor_SMD:R_0603_1608Metric
- R11: renamed from R5; footprint Resistor_SMD:R_0603_1608Metric_Pad0.98x0.95mm_HandSolder -> Resistor_SMD:R_0603_1608Metric
- R12: renamed from R2; footprint Resistor_SMD:R_0603_1608Metric_Pad0.98x0.95mm_HandSolder -> Resistor_SMD:R_0603_1608Metric
- R13: renamed from R1; footprint Resistor_SMD:R_0603_1608Metric_Pad0.98x0.95mm_HandSolder -> Resistor_SMD:R_0603_1608Metric
- R14: renamed from R3; footprint Resistor_SMD:R_0603_1608Metric_Pad0.98x0.95mm_HandSolder -> Resistor_SMD:R_0603_1608Metric
- R15: renamed from R4; footprint Resistor_SMD:R_0603_1608Metric_Pad0.98x0.95mm_HandSolder -> Resistor_SMD:R_0603_1608Metric
- R16: renamed from R14; footprint Resistor_SMD:R_0603_1608Metric_Pad0.98x0.95mm_HandSolder -> Resistor_SMD:R_0603_1608Metric
- R17: renamed from R15; footprint Resistor_SMD:R_0603_1608Metric_Pad0.98x0.95mm_HandSolder -> Resistor_SMD:R_0603_1608Metric
- R18: renamed from R16; footprint Resistor_SMD:R_0603_1608Metric_Pad0.98x0.95mm_HandSolder -> Resistor_SMD:R_0603_1608Metric
- R19: renamed from R17; footprint Resistor_SMD:R_0603_1608Metric_Pad0.98x0.95mm_HandSolder -> Resistor_SMD:R_0603_1608Metric
- R2: renamed from R11; footprint Resistor_SMD:R_0603_1608Metric_Pad0.98x0.95mm_HandSolder -> Resistor_SMD:R_0603_1608Metric
- R20: renamed from R18; footprint Resistor_SMD:R_0603_1608Metric_Pad0.98x0.95mm_HandSolder -> Resistor_SMD:R_0603_1608Metric
- R21, R6, R7: footprint Resistor_SMD:R_0603_1608Metric_Pad0.98x0.95mm_HandSolder -> Resistor_SMD:R_0603_1608Metric
- R3: renamed from R12; footprint Resistor_SMD:R_0603_1608Metric_Pad0.98x0.95mm_HandSolder -> Resistor_SMD:R_0603_1608Metric
- R4: renamed from R13; footprint Resistor_SMD:R_0603_1608Metric_Pad0.98x0.95mm_HandSolder -> Resistor_SMD:R_0603_1608Metric
- R5: renamed from R19; footprint Resistor_SMD:R_0603_1608Metric_Pad0.98x0.95mm_HandSolder -> Resistor_SMD:R_0603_1608Metric
- R8: renamed from R20; footprint Resistor_SMD:R_0603_1608Metric_Pad0.98x0.95mm_HandSolder -> Resistor_SMD:R_0603_1608Metric
- R9: renamed from R8; footprint Resistor_SMD:R_0603_1608Metric_Pad0.98x0.95mm_HandSolder -> Resistor_SMD:R_0603_1608Metric
- TP4: value TestPoint -> TX
- TP5: value TestPoint -> RX
- Y1: renamed from Y2; footprint Crystal:Crystal_SMD_3225-4Pin_3.2x2.5mm_HandSoldering -> Crystal:Crystal_SMD_3225-4Pin_3.2x2.5mm
- renumbered J2 to J1, J3 to J2, U2 to U5, U3 to U6
Connections:
- net +3V3: now also J3.1 (VCC), U2.2 (VO), U3.1 (VBAT), U3.24 (VDD), U3.36 (VDD), U3.40 (PB4), U3.41 (PB5), U3.42 (PB6), U3.48 (VDD), U3.9 (VDDA)
- net +5V: now also U1.5 (VBUS), U2.3 (VI)
- net GND: now also J3.5 (GND), J4.3 (GND), J4.5 (GND), J4.9 (GNDDetect), TP6.1, U1.2 (GND), U2.1 (GND), U3.23 (VSS), U3.35 (VSS), U3.44 (BOOT0), U3.47 (VSS), U3.8 (VSSA)
- net LED0: now also U3.20 (PB2)
- net LED1: now also U3.21 (PB10)
- net LED2: now also U3.22 (PB11)
- net NRST: now also J3.3 (~{RESET}), U3.7 (NRST)
- net RST: now also U3.12 (PA2)
- net RST_SENSE: now also U3.17 (PA7)
- net USBX1+: now also U1.4 (I/O2)
- net USBX1-: now also U1.6 (I/O1)
- net USBX2+: now also U3.33 (PA12)
- net USBX2-: now also U3.32 (PA11)
- net VREF: now also J4.1 (VTref)
- net at J1.A7 (D-), J1.B7 (D-): now also U1.1 (I/O1)
- net at J1.A6 (D+), J1.B6 (D+): now also U1.3 (I/O2)
- net at C1.1, R3.2, R4.1: now also U3.18 (PB0)
- net at U6.2 (1A): now also U3.14 (PA4)
- net at U6.5 (DIR): now also U3.11 (PA1)
- net at R1.2, R2.1: now also U3.26 (PB13)
- net at TP3.1: now also U3.43 (PB7)
- net at R14.2: now also J4.6 (SWO/TDO)
- net at TP1.1: now also U3.19 (PB1)
- net at U5.2 (1A): now also U3.16 (PA6)
- net at R11.2: now also J4.10 (~{RESET})
- net at R13.2: now also J4.2 (SWDIO/TMS)
- net at R12.2: now also J4.4 (SWCLK/TCK)
- net at R15.2: now also J4.8 (NC/TDI)
- net at U4.2 (1A): now also U3.15 (PA5)
- net at U4.3 (2A): now also U3.13 (PA3)
- net at C3.2, Y1.1: now also U3.6 (PD1)
- net at J2.1 (Pin_1), R5.2: now also U3.25 (PB12)
- net TX: now reaches TP4.1
- net TX: now also U3.30 (PA9)
- net at C2.1, Y1.3: now also U3.5 (PD0)
- net at TP2.1: now also U3.39 (PB3)
- net at R8.1: now also U3.29 (PA8)
- net RX: now reaches TP5.1
- net RX: now also U3.31 (PA10)
- new net SWCLK: J3.4 (SWCLK), U3.37 (PA14)
- new net SWDIO: J3.2 (SWDIO), U3.34 (PA13)
- no-connect marks 13 -> 14
Other:
- note removed: "C9002"
- note removed: "NCP698SQ33T1G"
- moved on the sheet: C4

Commit message: bom, schematic, drc corrections and add logo
Parts:
- C4: LCSC Part C15849 -> C19702
- C5: LCSC Part C15849 -> C86295
- J4: LCSC Part (none) -> C42372555
- R11, R12, R13, R14, R15, R16: LCSC Part C105588 -> C105588
- U1: LCSC Part (none) -> C2827654
- U2: LCSC Part (none) -> C460428
- U3: LCSC Part (none) -> C8304
- Y1: LCSC Part C9002 -> C2682775
Other:
- note added: "Based on: https://github.com/blackmagic-debug/black-magic-org/blob/main/_assets/bmpm_v2_1e_schematic.pdf"
- note added: "Black Smoke Probe"
- note added: "Cortex Connector"
- note added: "Level Shifter"
- note added: "MCU"
- note added: "Status LEDs"
- note added: "USB"
- note added: "Voltage Regulator"
- company: (none) -> @casartar
- moved on the sheet: C4, C5, J1, R6, R7, U1, U2
