File: Black-Smoke-Probe.kicad_sch (KiCad schematic)
At the start: 59 parts, among them J1 USB_C_Receptacle_USB2.0_14P, J2 MCU_BOOT, J3 SWD_TagConnect, J4 Conn_ARM_JTAG_SWD_10, U1 USBLC6-2SC6, U2 AZ1117-3.3, U3 STM32F103CBTx, U4 74LVC2T45DC, U5 74LVC2T45DC, U6 74LVC2T45DC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

Commit message: v1.1.1 changed capacitor from 100nf to 30pf
Parts:
- C3: value 100nF -> 30pF; LCSC Part C14663 -> C1658
- C4: LCSC Part C19702 -> C19702
- C5: LCSC Part C86295 -> C86295
- Y1: LCSC Part C2682775 -> C2682775
Changed lines of the file:
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@@
 	(title_block
 		(title "Black-Smoke-Probe")
-		(date "2025-04-05")
-		(rev "v1.1")
+		(date "2025-04-14")
+		(rev "v1.1.1")
 		(company "@casartar")
 		(comment 1 "License: CC-BY-SA 4.0")
@@
 			)
 		)
-		(property "LCSC Part" " C19702"
+		(property "LCSC Part" "C19702"
 			(at 66.675 81.915 0)
 			(effects
@@
 			)
 		)
-		(property "Value" "100nF"
+		(property "Value" "30pF"
 			(at 35.56 129.54 90)
 			(effects
@@
 			)
 		)
-		(property "LCSC Part" "C14663 "
+		(property "LCSC Part" "C1658 "
 			(at 27.94 127 0)
 			(effects
@@
 			)
 		)
-		(property "LCSC Part" " C2682775"
+		(property "LCSC Part" "C2682775"
 			(at 31.75 121.92 0)
 			(effects
@@
 			)
 		)
-		(property "LCSC Part" " C86295"
+		(property "LCSC Part" "C86295"
 			(at 88.265 81.915 0)
 			(effects
